Commit message: Update the soccer_nao.urdf to use the new Nao meshes path.

File: robocup_model_resources/nao_models/nao_soccer/nao_simple_shapes.urdf (robot description, URDF)
Before this commit: robot naoH25V40, 76 links, 75 joints
Links:
- link Head: geometry collision cylinder length=0.14 radius=0.04; visual mesh filename=package://nao_meshes/meshes/V40/HeadPitch.dae scale=0.1 0.1 0.1
- link LBicep: geometry collision cylinder length=0.09 radius=0.02; visual mesh filename=package://nao_meshes/meshes/V40/LShoulderRoll.dae scale=0.1 0.1 0.1
- link LFinger11: geometry visual mesh filename=package://nao_meshes/meshes/V40/LFinger11.dae scale=0.1 0.1 0.1
- link LFinger12: geometry visual mesh filename=package://nao_meshes/meshes/V40/LFinger12.dae scale=0.1 0.1 0.1
- link LFinger13: geometry visual mesh filename=package://nao_meshes/meshes/V40/LFinger13.dae scale=0.1 0.1 0.1
- link LFinger21: geometry visual mesh filename=package://nao_meshes/meshes/V40/LFinger21.dae scale=0.1 0.1 0.1
- link LFinger22: geometry visual mesh filename=package://nao_meshes/meshes/V40/LFinger22.dae scale=0.1 0.1 0.1
- link LFinger23: geometry visual mesh filename=package://nao_meshes/meshes/V40/LFinger23.dae scale=0.1 0.1 0.1
- link LForeArm: geometry collision cylinder length=0.05065 radius=0.02; visual mesh filename=package://nao_meshes/meshes/V40/LElbowRoll.dae scale=0.1 0.1 0.1
- link LHip: geometry visual mesh filename=package://nao_meshes/meshes/V40/LHipRoll.dae scale=0.1 0.1 0.1
- link LPelvis: geometry visual mesh filename=package://nao_meshes/meshes/V40/LHipYawPitch.dae scale=0.1 0.1 0.1
- link LShoulder: geometry visual mesh filename=package://nao_meshes/meshes/V40/LShoulderPitch.dae scale=0.1 0.1 0.1
- link LThigh: geometry collision cylinder length=0.1 radius=0.04; visual mesh filename=package://nao_meshes/meshes/V40/LHipPitch.dae scale=0.1 0.1 0.1
- link LThumb1: geometry visual mesh filename=package://nao_meshes/meshes/V40/LThumb1.dae scale=0.1 0.1 0.1
- link LThumb2: geometry visual mesh filename=package://nao_meshes/meshes/V40/LThumb2.dae scale=0.1 0.1 0.1
- link LTibia: geometry collision cylinder length=0.1 radius=0.04; visual mesh filename=package://nao_meshes/meshes/V40/LKneePitch.dae scale=0.1 0.1 0.1
- link Neck: geometry visual mesh filename=package://nao_meshes/meshes/V40/HeadYaw.dae scale=0.1 0.1 0.1
- link RBicep: geometry collision cylinder length=0.09 radius=0.02; visual mesh filename=package://nao_meshes/meshes/V40/RShoulderRoll.dae scale=0.1 0.1 0.1
- link RFinger11: geometry visual mesh filename=package://nao_meshes/meshes/V40/RFinger11.dae scale=0.1 0.1 0.1
- link RFinger12: geometry visual mesh filename=package://nao_meshes/meshes/V40/RFinger12.dae scale=0.1 0.1 0.1
- link RFinger13: geometry visual mesh filename=package://nao_meshes/meshes/V40/RFinger13.dae scale=0.1 0.1 0.1
- link RFinger21: geometry visual mesh filename=package://nao_meshes/meshes/V40/RFinger21.dae scale=0.1 0.1 0.1
- link RFinger22: geometry visual mesh filename=package://nao_meshes/meshes/V40/RFinger22.dae scale=0.1 0.1 0.1
- link RFinger23: geometry visual mesh filename=package://nao_meshes/meshes/V40/RFinger23.dae scale=0.1 0.1 0.1
- link RForeArm: geometry collision cylinder length=0.05065 radius=0.02; visual mesh filename=package://nao_meshes/meshes/V40/RElbowRoll.dae scale=0.1 0.1 0.1
- link RHip: geometry visual mesh filename=package://nao_meshes/meshes/V40/RHipRoll.dae scale=0.1 0.1 0.1
- link RPelvis: geometry collision cylinder length=0.1 radius=0.04; visual mesh filename=package://nao_meshes/meshes/V40/RHipYawPitch.dae scale=0.1 0.1 0.1
- link RShoulder: geometry visual mesh filename=package://nao_meshes/meshes/V40/RShoulderPitch.dae scale=0.1 0.1 0.1
- link RThigh: geometry visual mesh filename=package://nao_meshes/meshes/V40/RHipPitch.dae scale=0.1 0.1 0.1
- link RThumb1: geometry visual mesh filename=package://nao_meshes/meshes/V40/RThumb1.dae scale=0.1 0.1 0.1
- link RThumb2: geometry visual mesh filename=package://nao_meshes/meshes/V40/RThumb2.dae scale=0.1 0.1 0.1
- link RTibia: geometry collision cylinder length=0.1 radius=0.04; visual mesh filename=package://nao_meshes/meshes/V40/RKneePitch.dae scale=0.1 0.1 0.1
- link l_ankle: geometry visual mesh filename=package://nao_meshes/meshes/V40/LAnklePitch.dae scale=0.1 0.1 0.1
- link l_sole: geometry collision box size=0.16 0.085 0.015; visual mesh filename=package://nao_meshes/meshes/V40/LAnkleRoll.dae scale=0.1 0.1 0.1
- link l_wrist: geometry collision box size=0.06 0.04 0.058; visual mesh filename=package://nao_meshes/meshes/V40/LWristYaw.dae scale=0.1 0.1 0.1
- link r_ankle: geometry visual mesh filename=package://nao_meshes/meshes/V40/RAnklePitch.dae scale=0.1 0.1 0.1
- link r_sole: geometry collision box size=0.16 0.085 0.015; visual mesh filename=package://nao_meshes/meshes/V40/RAnkleRoll.dae scale=0.1 0.1 0.1
- link r_wrist: geometry collision box size=0.06 0.04 0.058; visual mesh filename=package://nao_meshes/meshes/V40/RWristYaw.dae scale=0.1 0.1 0.1
- link torso: geometry collision box size=0.1 0.1 0.2115; visual mesh filename=package://nao_meshes/meshes/V40/Torso.dae scale=0.1 0.1 0.1
